File: kicad_tr2023/backlamp.kicad_sch (KiCad schematic)
At the start: 5 parts

Commit message: sync chg
Parts:
- J?: value BACKLAMP -> LAMP
- J?: value Arduino_A7 -> A7
Changed lines of the file:
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@@
     (in_bom yes) (on_board yes) (fields_autoplaced)
     (property "Reference" "J?" (id 0) (at 41.529 49.53 0))
-    (property "Value" "BACKLAMP" (id 1) (at 41.529 52.07 0))
+    (property "Value" "LAMP" (id 1) (at 41.529 52.07 0))
     (property "Footprint" "Connector_PinHeader_2.54mm:PinHeader_1x02_P2.54mm_Vertical" (id 2) (at 40.894 55.372 0)
       (effects (font (size 1.27 1.27)) hide)
@@
   (symbol (lib_id "Connector:Conn_01x01_Male") (at 70.104 35.814 270) (unit 1)
     (in_bom yes) (on_board yes) (fields_autoplaced)
-    (property "Reference" "J?" (id 0) (at 71.374 35.1789 90)
+    (property "Reference" "J?" (id 0) (at 71.12 35.1789 90)
       (effects (font (size 1.27 1.27)) (justify left))
     )
-    (property "Value" "Arduino_A7" (id 1) (at 71.374 37.7189 90)
+    (property "Value" "A7" (id 1) (at 71.12 37.7189 90)
       (effects (font (size 1.27 1.27)) (justify left))
     )
