File: kicad_tr2023/driver.kicad_sch (KiCad schematic)
At the start: 7 parts, among them J14 Arduino_D10, J15 Conn_FET, U1 MIC4427

Commit message: sync chg
Parts:
- removed D1: FR107, Diode_THT:D_DO-41_SOD81_P10.16mm_Horizontal, symbol Diode:1N4007
Connections:
- net at R1.2, U1.2 (IN_A): now also J14.1 (Pin_1)
Changed lines of the file:
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@@
-    (stroke (width 0) (type default) (color 0 0 0 0))
-  )
-  (wire (pts (xy 88.9 68.326) (xy 84.074 68.326))
     (stroke (width 0) (type default) (color 0 0 0 0))
   )
@@
     (stroke (width 0) (type default) (color 0 0 0 0))
   )
-  (wire (pts (xy 73.914 68.326) (xy 76.454 68.326))
+  (wire (pts (xy 73.914 68.326) (xy 88.9 68.326))
     (stroke (width 0) (type default) (color 0 0 0 0))
   )
@@
       (effects (font (size 1.27 1.27)) hide)
     )
-    (pin "1")
-    (pin "2")
-  )
-  (symbol (lib_id "Diode:1N4007") (at 80.264 68.326 180) (unit 1)
-    (in_bom yes) (on_board yes) (fields_autoplaced)
-    (property "Reference" "D1" (id 0) (at 80.264 61.976 0))
-    (property "Value" "FR107" (id 1) (at 80.264 64.516 0))
-    (property "Footprint" "Diode_THT:D_DO-41_SOD81_P10.16mm_Horizontal" (id 2) (at 80.264 63.881 0)
-      (effects (font (size 1.27 1.27)) hide)
-    )
-    (property "Datasheet" "http://www.vishay.com/docs/88503/1n4001.pdf" (id 3) (at 80.264 68.326 0)
-      (effects (font (size 1.27 1.27)) hide)
-    )

Commit message: pre
Parts:
- added R?: 10, Resistor_THT:R_Axial_DIN0207_L6.3mm_D2.5mm_P10.16mm_Horizontal, symbol Device:R
Connections:
- net at J15.1 (Pin_1), R11.1: now also R?.1
- net at R11.2, U1.7 (OUT_A): now also R?.2
Other:
- moved on the sheet: J15
Changed lines of the file:
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@@
   (junction (at 97.79 83.82) (diameter 0) (color 0 0 0 0)
   )
+  (junction (at 126.492 68.326) (diameter 0) (color 0 0 0 0)
+  )
   (junction (at 88.9 68.326) (diameter 0) (color 0 0 0 0)
   )
@@
   )
   (junction (at 88.9 83.82) (diameter 0) (color 0 0 0 0)
+  )
+  (junction (at 140.97 68.326) (diameter 0) (color 0 0 0 0)
   )
   (no_connect (at 123.444 73.406))
@@
     (stroke (width 0) (type default) (color 0 0 0 0))
   )
+  (wire (pts (xy 140.97 68.326) (xy 147.574 68.326))
+    (stroke (width 0) (type default) (color 0 0 0 0))
+  )
   (wire (pts (xy 65.024 83.82) (xy 65.024 88.646))
     (stroke (width 0) (type default) (color 0 0 0 0))
@@
     (stroke (width 0) (type default) (color 0 0 0 0))
   )
+  (wire (pts (xy 126.492 62.738) (xy 126.492 68.326))
+    (stroke (width 0) (type default) (color 0 0 0 0))
+  )
+  (wire (pts (xy 126.492 68.326) (xy 129.54 68.326))
+    (stroke (width 0) (type default) (color 0 0 0 0))
+  )
   (wire (pts (xy 103.124 73.406) (xy 97.79 73.406))
     (stroke (width 0) (type default) (color 0 0 0 0))
@@
     (stroke (width 0) (type default) (color 0 0 0 0))
   )
-  (wire (pts (xy 137.16 68.326) (xy 142.24 68.326))
+  (wire (pts (xy 137.16 68.326) (xy 140.97 68.326))
     (stroke (width 0) (type default) (color 0 0 0 0))
   )
@@
     (stroke (width 0) (type default) (color 0 0 0 0))
   )
+  (wire (pts (xy 129.54 62.738) (xy 126.492 62.738))
+    (stroke (width 0) (type default) (color 0 0 0 0))
+  )
   (wire (pts (xy 88.9 68.326) (xy 103.124 68.326))
     (stroke (width 0) (type default) (color 0 0 0 0))
@@
     (stroke (width 0) (type default) (color 0 0 0 0))
   )
-  (wire (pts (xy 123.444 68.326) (xy 129.54 68.326))
+  (wire (pts (xy 123.444 68.326) (xy 126.492 68.326))
+    (stroke (width 0) (type default) (color 0 0 0 0))
+  )
+  (wire (pts (xy 140.97 62.738) (xy 140.97 68.326))
+    (stroke (width 0) (type default) (color 0 0 0 0))
+  )
+  (wire (pts (xy 137.16 62.738) (xy 140.97 62.738))
     (stroke (width 0) (type default) (color 0 0 0 0))
   )
@@
     (pin "1")
   )
-  (symbol (lib_id "Connector:Conn_01x01_Male") (at 142.24 63.246 270) (unit 1)
+  (symbol (lib_id "Connector:Conn_01x01_Male") (at 147.574 63.246 270) (unit 1)
     (in_bom yes) (on_board yes)
-    (property "Reference" "J15" (id 0) (at 147.066 63.881 0))
-    (property "Value" "Conn_FET" (id 1) (at 144.526 63.881 0))
-    (property "Footprint" "Connector_PinHeader_2.54mm:PinHeader_1x01_P2.54mm_Vertical" (id 2) (at 142.24 63.246 0)
-      (effects (font (size 1.27 1.27)) hide)
-    )
-    (property "Datasheet" "~" (id 3) (at 142.24 63.246 0)
+    (property "Reference" "J15" (id 0) (at 152.4 63.881 0))
+    (property "Value" "Conn_FET" (id 1) (at 149.86 63.881 0))
+    (property "Footprint" "Connector_PinHeader_2.54mm:PinHeader_1x01_P2.54mm_Vertical" (id 2) (at 147.574 63.246 0)
+      (effects (font (size 1.27 1.27)) hide)
+    )
+    (property "Datasheet" "~" (id 3) (at 147.574 63.246 0)
       (effects (font (size 1.27 1.27)) hide)
     )
@@
     (pin "1")
   )
+  (symbol (lib_id "Device:R") (at 133.35 62.738 270) (unit 1)
+    (in_bom yes) (on_board yes) (fields_autoplaced)
+    (property "Reference" "R?" (id 0) (at 133.35 56.642 90))
+    (property "Value" "10" (id 1) (at 133.35 59.182 90))
+    (property "Footprint" "Resistor_THT:R_Axial_DIN0207_L6.3mm_D2.5mm_P10.16mm_Horizontal" (id 2) (at 133.35 60.96 90)
+      (effects (font (size 1.27 1.27)) hide)
+    )
+    (property "Datasheet" "" (id 3) (at 133.35 62.738 0)
+      (effects (font (size 1.27 1.27)) hide)
+    )
+    (pin "1")
+    (pin "2")
+  )
 )
