File: kicad_tr2023/kicad_tr2023.kicad_sch (KiCad schematic)
At the start: 0 parts

Commit message: sync chg
Other:
- added sheet backlamp (backlamp.kicad_sch)
Changed lines of the file:
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@@
+    )
+  )
+  (sheet (at 217.932 133.096) (size 16.002 8.382) (fields_autoplaced)
+    (stroke (width 0.1524) (type solid) (color 0 0 0 0))
+    (fill (color 0 0 0 0.0000))
+    (property "Sheet name" "backlamp" (id 0) (at 217.932 132.3844 0)
+      (effects (font (size 1.27 1.27)) (justify left bottom))
+    )
+    (property "Sheet file" "backlamp.kicad_sch" (id 1) (at 217.932 142.0626 0)
+      (effects (font (size 1.27 1.27)) (justify left top))
     )
   )
@@
     (path "/0ce664fb-5e27-4cb3-9bd5-32578bb2d300" (page "4"))
     (path "/34d45c12-9ce4-4b51-aaf8-d1ea918f268a" (page "5"))
+    (path "/b9f9b85b-4028-4ab4-b5d9-32a450460432" (page "6"))
   )
   (symbol_instances
@@
       (reference "#PWR0102") (unit 1) (value "+5V") (footprint "")
     )
+    (path "/b9f9b85b-4028-4ab4-b5d9-32a450460432/93039435-bc3f-4db4-93c5-5d2a91d46fa3"
+      (reference "#PWR?") (unit 1) (value "GND") (footprint "")
+    )
+    (path "/b9f9b85b-4028-4ab4-b5d9-32a450460432/adc5dabe-4e2e-4deb-8249-d4e16c17bdd3"
+      (reference "#PWR?") (unit 1) (value "VCC") (footprint "")
+    )
     (path "/71204b6c-b957-415d-b644-1807de96873a/a619ab21-6b84-41fa-a08d-61b36e21f87a"
       (reference "C5") (unit 1) (value "475") (footprint "Capacitor_THT:C_Disc_D3.0mm_W2.0mm_P2.50mm")
@@
       (reference "C9") (unit 1) (value "6.8n") (footprint "Capacitor_THT:C_Disc_D3.0mm_W2.0mm_P2.50mm")
     )
-    (path "/c32b5ce1-bf46-41e2-af6e-64b1984d359d/086301b8-30d2-493c-b5b7-91a084452c95"
-      (reference "D1") (unit 1) (value "FR107") (footprint "Diode_THT:D_DO-41_SOD81_P10.16mm_Horizontal")
+    (path "/b9f9b85b-4028-4ab4-b5d9-32a450460432/b5f90935-fc27-424b-91cd-0e83283affd4"
+      (reference "C?") (unit 1) (value "100n") (footprint "Capacitor_THT:C_Disc_D5.0mm_W2.5mm_P2.50mm")
     )
     (path "/71204b6c-b957-415d-b644-1807de96873a/122ee31d-cc4b-4a2f-95aa-857731f4d9be"
@@
       (reference "J16") (unit 1) (value "Arduino_D2") (footprint "Connector_PinHeader_2.54mm:PinHeader_1x01_P2.54mm_Vertical")
     )
+    (path "/b9f9b85b-4028-4ab4-b5d9-32a450460432/0d0531a3-7e72-42ab-b9e6-147bc805eb73"
+      (reference "J?") (unit 1) (value "LAMP") (footprint "Connector_PinHeader_2.54mm:PinHeader_1x02_P2.54mm_Vertical")
+    )
+    (path "/b9f9b85b-4028-4ab4-b5d9-32a450460432/dd74102a-157f-4f5c-8d97-c6f9a9173dc7"
+      (reference "J?") (unit 1) (value "A7") (footprint "Connector_PinHeader_2.54mm:PinHeader_1x01_P2.54mm_Vertical")
+    )
     (path "/c32b5ce1-bf46-41e2-af6e-64b1984d359d/017ab7d7-a720-4b3f-882c-681606e828ef"
       (reference "R1") (unit 1) (value "10K") (footprint "Resistor_THT:R_Axial_DIN0207_L6.3mm_D2.5mm_P10.16mm_Horizontal")
@@
       (reference "R14") (unit 1) (value "1K") (footprint "Resistor_THT:R_Axial_DIN0207_L6.3mm_D2.5mm_P7.62mm_Horizontal")
     )
+    (path "/b9f9b85b-4028-4ab4-b5d9-32a450460432/9c82e11d-9699-435a-8eca-b4ab8ac28975"
+      (reference "R?") (unit 1) (value "150K") (footprint "Resistor_THT:R_Axial_DIN0207_L6.3mm_D2.5mm_P7.62mm_Horizontal")
+    )
+    (path "/b9f9b85b-4028-4ab4-b5d9-32a450460432/a09c60f2-aeba-4fb5-824c-fd20a73713e3"
+      (reference "R?") (unit 1) (value "10K") (footprint "Resistor_THT:R_Axial_DIN0207_L6.3mm_D2.5mm_P7.62mm_Horizontal")
+    )
     (path "/71204b6c-b957-415d-b644-1807de96873a/2574d129-1724-457e-808e-650e7ac2a7f1"

Commit message: pre
Parts:
- added C1, C4, C5: 100n, Capacitor_THT:C_Disc_D3.0mm_W2.0mm_P2.50mm, symbol Device:C
- added C2: 10n, Capacitor_THT:C_Disc_D3.0mm_W2.0mm_P2.50mm, symbol Device:C
- added C3: 6.8n, Capacitor_THT:C_Disc_D3.0mm_W2.0mm_P2.50mm, symbol Device:C
- added C6: 1u, Capacitor_THT:C_Disc_D3.0mm_W2.0mm_P2.50mm, symbol Device:C
- added C7: 4.7u, Capacitor_THT:C_Disc_D3.0mm_W2.0mm_P2.50mm, symbol Device:C
- added C8: 100n, Capacitor_THT:C_Disc_D5.0mm_W2.5mm_P2.50mm, symbol Device:C
- added J1: Conn_VIN, Connector_PinHeader_2.54mm:PinHeader_1x01_P2.54mm_Vertical, symbol Connector:Conn_01x01_Male
- added J2: Conn_GND, Connector_PinHeader_2.54mm:PinHeader_1x01_P2.54mm_Vertical, symbol Connector:Conn_01x01_Male
- added J3: Arduino_D2, Connector_PinHeader_2.54mm:PinHeader_1x01_P2.54mm_Vertical, symbol Connector:Conn_01x01_Male
- added J4: Arduino_D10, Connector_PinHeader_2.54mm:PinHeader_1x01_P2.54mm_Vertical, symbol Connector:Conn_01x01_Male
- added J5: Conn_ACCEL, Connector:FanPinHeader_1x03_P2.54mm_Vertical, symbol Connector:Conn_01x03_Male
- added J6: Arduino_A6, Connector_PinHeader_2.54mm:PinHeader_1x01_P2.54mm_Vertical, symbol Connector:Conn_01x01_Male
- added J7: Conn_FET, Connector_PinHeader_2.54mm:PinHeader_1x01_P2.54mm_Vertical, symbol Connector:Conn_01x01_Male
- added J8: LAMP, Connector_PinHeader_2.54mm:PinHeader_1x02_P2.54mm_Vertical, symbol Connector:Conn_01x02_Male
- added J9: A7, Connector_PinHeader_2.54mm:PinHeader_1x01_P2.54mm_Vertical, symbol Connector:Conn_01x01_Male
- added R1, R5: 330, Resistor_THT:R_Axial_DIN0207_L6.3mm_D2.5mm_P10.16mm_Horizontal, symbol Device:R
- added R10: 150K, Resistor_THT:R_Axial_DIN0207_L6.3mm_D2.5mm_P7.62mm_Horizontal, symbol Device:R
- added R11: 10K, Resistor_THT:R_Axial_DIN0207_L6.3mm_D2.5mm_P7.62mm_Horizontal, symbol Device:R
- added R2: 470, Resistor_THT:R_Axial_DIN0207_L6.3mm_D2.5mm_P10.16mm_Horizontal, symbol Device:R
- added R3, R4, R7: 1K, Resistor_THT:R_Axial_DIN0207_L6.3mm_D2.5mm_P10.16mm_Horizontal, symbol Device:R
- added R6: 10K, Resistor_THT:R_Axial_DIN0207_L6.3mm_D2.5mm_P10.16mm_Horizontal, symbol Device:R
- added R8, R9: 10, Resistor_THT:R_Axial_DIN0207_L6.3mm_D2.5mm_P10.16mm_Horizontal, symbol Device:R
- added RV1: 5K, Potentiometer_THT:Potentiometer_ACP_CA9-V10_Vertical, symbol Device:R_Potentiometer
- added RV2: 20K, Potentiometer_THT:Potentiometer_ACP_CA9-V10_Vertical, symbol Device:R_Potentiometer
- added U1: LM317_TO-220, Package_TO_SOT_THT:TO-220-3_Vertical, symbol Regulator_Linear:LM317_TO-220
- added U2: NE555P, Package_DIP:DIP-8_W7.62mm, symbol Timer:NE555P
- added U3: LM358, Package_DIP:DIP-8_W7.62mm, symbol Amplifier_Operational:TL072
- added U4: TL431LP, Package_TO_SOT_THT:TO-92L_Wide, symbol Reference_Voltage:TL431LP
- added U5: MIC4427, Package_DIP:DIP-8_W7.62mm, symbol Driver_FET:MIC4427
Connections:
- new net: C7.1, RV2.2, U3.3 (+)
- new net: C2.2, U2.5 (CV)
- new net: R5.1, R6.2, U5.2 (IN_A)
- new net: R8.2, R9.2, U5.7 (OUT_A)
- new net: C4.1, R1.1, R2.2, U1.1 (ADJ)
- new net: C5.1, R1.2, RV1.2, RV1.3, U1.2 (VO), U3.8 (V+)
- new net: J5.1 (Pin_1), RV1.1, RV2.1, U4.1 (REF), U4.3 (K)
- new net: C3.2, R4.1, U2.2 (TR), U2.6 (THR)
- new net: R3.1, R4.2, U2.7 (DIS)
- new net: J4.1 (Pin_1), R5.2
- new net: J7.1 (Pin_1), R8.1, R9.1
- new net: J6.1 (Pin_1), R7.2, U3.1, U3.2 (-)
- new net A7: C8.1, J9.1 (Pin_1), R10.1, R11.2
- new net D2: J3.1 (Pin_1), U2.3 (Q)
- new net GND: C1.2, C2.1, C3.1, C4.2, C5.2, C6.2, C7.2, C8.2, J2.1 (Pin_1), J5.3 (Pin_3), J8.2 (Pin_2), R11.1, R2.1, R6.1, R7.1, RV2.3, U2.1 (GND), U3.4 (V-), U4.2 (A), U5.3 (GND), U5.4 (IN_B)
- new net VCC: C6.1, J8.1 (Pin_1), R10.2, U5.6 (V+)
- new net VIN_BULK: C1.1, J1.1 (Pin_1), R3.2, U1.3 (VI), U2.8 (VCC)
- no-connect marks 0 -> 6
Other:
- removed sheet accel
- removed sheet backlamp
- removed sheet driver
- removed sheet generator
- note added: "ADC7"

Commit message: 202310
Parts:
- removed C1, C4, C5: 100n, Capacitor_THT:C_Disc_D3.0mm_W2.0mm_P2.50mm, symbol Device:C
- removed C8: 100n, Capacitor_THT:C_Disc_D5.0mm_W2.5mm_P2.50mm, symbol Device:C
- removed J1: Conn_VIN, Connector_PinHeader_2.54mm:PinHeader_1x01_P2.54mm_Vertical, symbol Connector:Conn_01x01_Male
- removed J8: LAMP, Connector_PinHeader_2.54mm:PinHeader_1x02_P2.54mm_Vertical, symbol Connector:Conn_01x02_Male
- removed J9: A7, Connector_PinHeader_2.54mm:PinHeader_1x01_P2.54mm_Vertical, symbol Connector:Conn_01x01_Male
- removed R1: 330, Resistor_THT:R_Axial_DIN0207_L6.3mm_D2.5mm_P10.16mm_Horizontal, symbol Device:R
- removed R2: 470, Resistor_THT:R_Axial_DIN0207_L6.3mm_D2.5mm_P10.16mm_Horizontal, symbol Device:R
- removed U1: LM317_TO-220, Package_TO_SOT_THT:TO-220-3_Vertical, symbol Regulator_Linear:LM317_TO-220
- added J10: Conn_FET_B, Connector_PinHeader_2.54mm:PinHeader_1x01_P2.54mm_Vertical, symbol Connector:Conn_01x01_Male
- added J11: REV_BTN, Connector_JST:JST_PH_B2B-PH-K_1x02_P2.00mm_Vertical, symbol Connector_Generic:Conn_01x02
- added J12: REV_SENS, Connector_PinHeader_2.54mm:PinHeader_1x01_P2.54mm_Vertical, symbol Connector:Conn_01x01_Male
- added J13: REV_CTRL, Connector_PinHeader_2.54mm:PinHeader_1x01_P2.54mm_Vertical, symbol Connector:Conn_01x01_Male
- added J14: REV_ACT, Connector_PinHeader_2.54mm:PinHeader_1x01_P2.54mm_Vertical, symbol Connector:Conn_01x01_Male
- added J4: PWM_B, Connector_PinHeader_2.54mm:PinHeader_1x01_P2.54mm_Vertical, symbol Connector:Conn_01x01_Male
- added J7: CONN_VCC, Connector_JST:JST_PH_B2B-PH-K_1x02_P2.00mm_Vertical, symbol Connector_Generic:Conn_01x02
- added J8: CONN_V3V5, Connector_JST:JST_PH_B2B-PH-K_1x02_P2.00mm_Vertical, symbol Connector_Generic:Conn_01x02
- added Q1: IPD50R380CE, Package_TO_SOT_SMD:TO-252-2, symbol Transistor_FET:IPD50R380CE
- added R12: 470, Resistor_THT:R_Axial_DIN0207_L6.3mm_D2.5mm_P10.16mm_Horizontal, symbol Device:R
- added R13, R14, R7: 10K, Resistor_THT:R_Axial_DIN0207_L6.3mm_D2.5mm_P10.16mm_Horizontal, symbol Device:R
- added R5: 330, Resistor_THT:R_Axial_DIN0207_L6.3mm_D2.5mm_P10.16mm_Horizontal, symbol Device:R
- C3: renamed from C7; footprint Capacitor_THT:C_Disc_D3.0mm_W2.0mm_P2.50mm -> Capacitor_THT:C_Disc_D7.0mm_W2.5mm_P5.00mm
- J1: renamed from J5; value Conn_ACCEL -> ACCEL_CTRL
- J2: renamed from J3; value Arduino_D2 -> GEN
- J3: renamed from J4; value Arduino_D10 -> PWM_A
- J5: renamed from J6; value Arduino_A6 -> ACCEL_SENS
- J9: renamed from J7; value Conn_FET -> Conn_FET_A
- R10: value 150K -> 10; footprint Resistor_THT:R_Axial_DIN0207_L6.3mm_D2.5mm_P7.62mm_Horizontal -> Resistor_THT:R_Axial_DIN0207_L6.3mm_D2.5mm_P10.16mm_Horizontal
- R11: value 10K -> 10; footprint Resistor_THT:R_Axial_DIN0207_L6.3mm_D2.5mm_P7.62mm_Horizontal -> Resistor_THT:R_Axial_DIN0207_L6.3mm_D2.5mm_P10.16mm_Horizontal
- renumbered C2 to C1, C3 to C2, C6 to C4, J2 to J6, R3 to R1, R4 to R2, R7 to R3, R5 to R4, U3 to U1, U4 to U3, U5 to U4
Connections:
- net GND: now also J7.2 (Pin_2), Q1.3 (S), R13.1, R14.1, R7.1; no longer R11.1, U4.4 (IN_B)
- net VCC: now also J7.1 (Pin_1); no longer R10.2
- net at U4.5 (OUT_B): now also R10.1, R11.1
- net +3V3: now reaches RV1.2, RV1.3, U1.8 (V+)
- net +3V3: now also J8.1 (Pin_1)
- net A7: no longer names the net of R11.2
- net A7: now also R10.2, J10.1 (Pin_1); no longer R10.1
- net D2: no longer names the net of J2.1 (Pin_1), U2.3 (Q)
- net VIN_BULK renamed +5V
- net +5V: now also J11.2 (Pin_2), J8.2 (Pin_2)
- new net: R5.1, R7.2, U4.4 (IN_B)
- new net: J13.1 (Pin_1), R12.1
- new net: Q1.1 (G), R12.2, R14.2
- new net: J4.1 (Pin_1), R5.2
- new net: J11.1 (Pin_1), J12.1 (Pin_1), R13.2
- new net: J14.1 (Pin_1), Q1.2 (D)
- no-connect marks 6 -> 5
Other:
- removed sheet reverse
- note added: "A6"
- note added: "D10"
- note added: "D2"
- note added: "D4"
- note added: "D5"
- note added: "D9"
- note removed: "ADC7"
- moved on the sheet: C1, C2, C3, C4, J1, J2, J3, J5, J6, J9, R1, R2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
